File: arduino-grove-beginner-kit/kicad/DHT-11.sch (KiCad schematic (older format))
At the start: 4 parts

Commit message: update circuits,
Parts:
- removed C?: C104,0805, Capacitor_SMD:C_0805_2012Metric_Pad1.15x1.40mm_HandSolder, symbol taobao-c:C104,0805
- removed J?: DHT-11, symbol taobao-components:DHT-11
- removed J?: Conn_01x04, symbol Connector_Generic:Conn_01x04
- removed R?: R472,0805, Resistor_SMD:R_0805_2012Metric_Pad1.15x1.40mm_HandSolder, symbol taobao-r:R472,0805
- added C? (x2): C106,0805, Capacitor_SMD:C_0805_2012Metric_Pad1.15x1.40mm_HandSolder, symbol taobao-c:C106,0805
- added C? (x3): C104,0805, Capacitor_SMD:C_0805_2012Metric_Pad1.15x1.40mm_HandSolder, symbol taobao-c:C104,0805
- added J? (x2): Conn_01x04, symbol Connector_Generic:Conn_01x04
- added Q? (x3): 2N7002, Package_TO_SOT_SMD:SOT-23, symbol Transistor_FET:2N7002
- added R? (x6): R472,0805, Resistor_SMD:R_0805_2012Metric_Pad1.15x1.40mm_HandSolder, symbol taobao-r:R472,0805
- added R? (x2): R0,0805, Resistor_SMD:R_0805_2012Metric_Pad1.15x1.40mm_HandSolder, symbol taobao-r:R0,0805
- added R? (x2): R103,0805, Resistor_SMD:R_0805_2012Metric_Pad1.15x1.40mm_HandSolder, symbol taobao-r:R103,0805
- added U?: LIS3DH, symbol taobao-components:LIS3DH
- added U?: XC6206P332MG-MR, symbol taobao-components:XC6206P332MG-MR
Connections:
- net GND: now also C?.1, C?.2, C?.2, C?.2, C?.2, J?.4 (Pin_4), R?.2, U?.1 (VSS), U?.10 (RES), U?.12 (GND), U?.5 (GND)
- new net: C?.2, U?.14 (VDD)
- new net: R?.1, U?.7 (SDO/SA0)
- new net: R?.1, U?.8 (CS)
- new net: Q?.2 (S), R?.2 (x3)
- new net: Q?.3 (D), R?.2 (x3)
- new net ADC1: J?.1 (Pin_1), U?.16 (ADC1)
- new net ADC2: J?.2 (Pin_2), U?.15 (ADC2)
- new net ADC3: J?.3 (Pin_3), U?.13 (ADC3)
- new net INT1: J?.4 (Pin_4), U?.11 (INT1)
- new net L_3V3: C?.1, C?.1, Q?.1 (G), Q?.1 (G), Q?.1 (G), R?.1, R?.1, R?.1, R?.2, U?.1 (VDD_IO), U?.2 (VOUT)
- new net L_SCK: R?.1
- new net L_SCL: U?.4 (SCL/SPC)
- new net L_SDA: R?.1, U?.6 (SDA/SDI/SDO)
- new net PC4_SDA: J?.2 (Pin_2), R?.2
- new net PC5_SCL: J?.1 (Pin_1), R?.2
- new net VCC: C?.1, C?.1, J?.3 (Pin_3), R?.1, R?.1, R?.1, U?.3 (VIN)
- no-connect marks 2 -> 1
