File: arduino-grove-beginner-kit/kicad/arduino-grove-beginner-kit.sch (KiCad schematic (older format))
At the start: 0 parts

Commit message: update circuits,
Changed lines of the file:
@@
 $Descr User 5846 4134
 encoding utf-8
-Sheet 1 3
+Sheet 1 4
 Title ""
 Date ""
@@
 F1 "DHT-11.sch" 50
 $EndSheet
+$Sheet
+S 2750 650  800  600
+U 5F3EA444
+F0 "sheet5F3EA444" 50
+F1 "DHT-11.sch" 50
+$EndSheet
