File: 7_by_9_breadboard-tryout/kicad/7_by_9_breadboard-tryout.kicad_pcb (KiCad board)
At the start: 2 copper layers, 2 parts

Commit message: update basically done,
Parts:
- removed R1: R103,0603, Resistor_SMD:R_0603_1608Metric_Pad1.05x0.95mm_HandSolder
- removed R2: R103,0805, Resistor_SMD:R_0805_2012Metric_Pad1.15x1.40mm_HandSolder
- added H1: MountingHole, footprint-lib:MountingHole_3.1mm_M3,rpi_like, F.Cu at (86.0, 66.0)
- added H2: MountingHole, footprint-lib:MountingHole_3.1mm_M3,rpi_like, F.Cu at (4.00, 4.00)
- added H3: MountingHole, footprint-lib:MountingHole_3.1mm_M3,rpi_like, F.Cu at (86.0, 4.00)
- added H4: MountingHole, footprint-lib:MountingHole_3.1mm_M3,rpi_like, F.Cu at (4.00, 66.0)
Other:
- board outline added: 90 x 70 mm
- board text added: "PCB breadboard 90 x 70"
Changed lines of the file:
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@@
-(kicad_pcb (version 20171130) (host pcbnew 5.1.5-52549c5~86~ubuntu18.04.1)
+(kicad_pcb (version 20171130) (host pcbnew 5.1.6-c6e7f7d~87~ubuntu18.04.1)
   (general
     (thickness 1.6)
-    (drawings 0)
+    (drawings 17)
     (tracks 0)
     (zones 0)
-    (modules 2)
+    (modules 4)
     (nets 1)
   )
-  (page A4)
+  (page User 148.488 105.004)
   (layers
     (0 F.Cu signal)
@@
     (uvia_dia 0.3)
     (uvia_drill 0.1)
-    (add_net "Net-(R1-Pad1)")
-    (add_net "Net-(R1-Pad2)")
-    (add_net "Net-(R2-Pad1)")
-    (add_net "Net-(R2-Pad2)")
   )
-  (module Resistor_SMD:R_0805_2012Metric_Pad1.15x1.40mm_HandSolder (layer F.Cu)
-    (at 25.2 23.27)
-    (descr "Resistor SMD 0805 (2012 Metric), square (rectangular) end terminal, IPC_7351 nominal with elongated pad for handsoldering. (Body size source: https://docs.google.com/spreadsheets/d/1BsfQQcO9C6DZCsRaXUlFlo91Tg2WpOkGARC1WS5S8t0/edit?usp=sharing), generated with kicad-footprint-generator")
-    (tags "resistor handsolder")
-    (attr smd)
-    (fp_text reference R2 (at 0 -1.65) (layer F.SilkS)
+  (module footprint-lib:MountingHole_3.1mm_M3,rpi_like locked (layer F.Cu)
+    (at 4 66)
+    (descr "Mounting Hole 2.7mm, no annular, M2.5")
+    (tags "mounting hole 2.7mm no annular m2.5")
+    (attr virtual)
+    (fp_text reference H4 (at 0 -3.7) (layer F.SilkS) hide
       (effects (font (size 1 1) (thickness 0.15)))
     )
-    (fp_text value R103,0805 (at 0 1.65) (layer F.Fab)
+    (fp_text value MountingHole (at 0 3.7) (layer F.Fab)
       (effects (font (size 1 1) (thickness 0.15)))
     )
-    (fp_text user %R (at 0 0) (layer F.Fab)
-      (effects (font (size 0.5 0.5) (thickness 0.08)))
-    )
-    (fp_line (start 1.85 0.95) (end -1.85 0.95) (layer F.CrtYd) (width 0.05))
-    (fp_line (start 1.85 -0.95) (end 1.85 0.95) (layer F.CrtYd) (width 0.05))
-    (fp_line (start -1.85 -0.95) (end 1.85 -0.95) (layer F.CrtYd) (width 0.05))
-    (fp_line (start -1.85 0.95) (end -1.85 -0.95) (layer F.CrtYd) (width 0.05))
-    (fp_line (start -0.261252 0.71) (end 0.261252 0.71) (layer F.SilkS) (width 0.12))
-    (fp_line (start -0.261252 -0.71) (end 0.261252 -0.71) (layer F.SilkS) (width 0.12))
-    (fp_line (start 1 0.6) (end -1 0.6) (layer F.Fab) (width 0.1))
-    (fp_line (start 1 -0.6) (end 1 0.6) (layer F.Fab) (width 0.1))
-    (fp_line (start -1 -0.6) (end 1 -0.6) (layer F.Fab) (width 0.1))
-    (fp_line (start -1 0.6) (end -1 -0.6) (layer F.Fab) (width 0.1))
-    (pad 2 smd roundrect (at 1.025 0) (size 1.15 1.4) (layers F.Cu F.Paste F.Mask) (roundrect_rratio 0.217391))
-    (pad 1 smd roundrect (at -1.025 0) (size 1.15 1.4) (layers F.Cu F.Paste F.Mask) (roundrect_rratio 0.217391))
-    (model ${KISYS3DMOD}/Resistor_SMD.3dshapes/R_0805_2012Metric.wrl
-      (at (xyz 0 0 0))
-      (scale (xyz 1 1 1))
-      (rotate (xyz 0 0 0))
-    )
+    (fp_circle (center 0 0) (end 1.905 0) (layer B.Mask) (width 1.2))
+    (fp_circle (center 0 0) (end 1.905 0) (layer F.Mask) (width 1.2))
+    (fp_circle (center 0 0) (end 2.95 0) (layer F.CrtYd) (width 0.05))
+    (fp_circle (center 0 0) (end 2.7 0) (layer Cmts.User) (width 0.15))
+    (pad "" np_thru_hole circle (at 0 0) (size 3.1 3.1) (drill 3.1) (layers *.Cu *.Mask)
+      (solder_mask_margin 1.5) (clearance 1.5))
   )
-  (module Resistor_SMD:R_0603_1608Metric_Pad1.05x0.95mm_HandSolder (layer F.Cu)
-    (at 25 26)
-    (descr "Resistor SMD 0603 (1608 Metric), square (rectangular) end terminal, IPC_7351 nominal with elongated pad for handsoldering. (Body size source: http://www.tortai-tech.com/upload/download/2011102023233369053.pdf), generated with kicad-footprint-generator")
-    (tags "resistor handsolder")
-    (attr smd)
-    (fp_text reference R1 (at 0 -1.43) (layer F.SilkS)
+  (module footprint-lib:MountingHole_3.1mm_M3,rpi_like locked (layer F.Cu)
+    (at 86 4)
+    (descr "Mounting Hole 2.7mm, no annular, M2.5")
+    (tags "mounting hole 2.7mm no annular m2.5")
+    (attr virtual)
+    (fp_text reference H3 (at 0 -3.7) (layer F.SilkS) hide
       (effects (font (size 1 1) (thickness 0.15)))
     )
-    (fp_text value R103,0603 (at 0 1.43) (layer F.Fab)
+    (fp_text value MountingHole (at 0 3.7) (layer F.Fab)
       (effects (font (size 1 1) (thickness 0.15)))
     )
-    (fp_text user %R (at 0 0) (layer F.Fab)
-      (effects (font (size 0.4 0.4) (thickness 0.06)))
+    (fp_circle (center 0 0) (end 1.905 0) (layer B.Mask) (width 1.2))
+    (fp_circle (center 0 0) (end 1.905 0) (layer F.Mask) (width 1.2))
+    (fp_circle (center 0 0) (end 2.95 0) (layer F.CrtYd) (width 0.05))
+    (fp_circle (center 0 0) (end 2.7 0) (layer Cmts.User) (width 0.15))
+    (pad "" np_thru_hole circle (at 0 0) (size 3.1 3.1) (drill 3.1) (layers *.Cu *.Mask)
+      (solder_mask_margin 1.5) (clearance 1.5))
+  )
+  (module footprint-lib:MountingHole_3.1mm_M3,rpi_like locked (layer F.Cu)
+    (at 4 4)
+    (descr "Mounting Hole 2.7mm, no annular, M2.5")
+    (tags "mounting hole 2.7mm no annular m2.5")
+    (attr virtual)
+    (fp_text reference H2 (at 0 -3.7) (layer F.SilkS) hide
+      (effects (font (size 1 1) (thickness 0.15)))
     )
-    (fp_line (start 1.65 0.73) (end -1.65 0.73) (layer F.CrtYd) (width 0.05))
-    (fp_line (start 1.65 -0.73) (end 1.65 0.73) (layer F.CrtYd) (width 0.05))
-    (fp_line (start -1.65 -0.73) (end 1.65 -0.73) (layer F.CrtYd) (width 0.05))
-    (fp_line (start -1.65 0.73) (end -1.65 -0.73) (layer F.CrtYd) (width 0.05))
-    (fp_line (start -0.171267 0.51) (end 0.171267 0.51) (layer F.SilkS) (width 0.12))
-    (fp_line (start -0.171267 -0.51) (end 0.171267 -0.51) (layer F.SilkS) (width 0.12))
-    (fp_line (start 0.8 0.4) (end -0.8 0.4) (layer F.Fab) (width 0.1))
-    (fp_line (start 0.8 -0.4) (end 0.8 0.4) (layer F.Fab) (width 0.1))
-    (fp_line (start -0.8 -0.4) (end 0.8 -0.4) (layer F.Fab) (width 0.1))
-    (fp_line (start -0.8 0.4) (end -0.8 -0.4) (layer F.Fab) (width 0.1))
-    (pad 2 smd roundrect (at 0.875 0) (size 1.05 0.95) (layers F.Cu F.Paste F.Mask) (roundrect_rratio 0.25))
-    (pad 1 smd roundrect (at -0.875 0) (size 1.05 0.95) (layers F.Cu F.Paste F.Mask) (roundrect_rratio 0.25))
-    (model ${KISYS3DMOD}/Resistor_SMD.3dshapes/R_0603_1608Metric.wrl
-      (at (xyz 0 0 0))
-      (scale (xyz 1 1 1))
-      (rotate (xyz 0 0 0))
+    (fp_text value MountingHole (at 0 3.7) (layer F.Fab)
+      (effects (font (size 1 1) (thickness 0.15)))
     )
+    (fp_circle (center 0 0) (end 1.905 0) (layer B.Mask) (width 1.2))
+    (fp_circle (center 0 0) (end 1.905 0) (layer F.Mask) (width 1.2))
+    (fp_circle (center 0 0) (end 2.95 0) (layer F.CrtYd) (width 0.05))
+    (fp_circle (center 0 0) (end 2.7 0) (layer Cmts.User) (width 0.15))
+    (pad "" np_thru_hole circle (at 0 0) (size 3.1 3.1) (drill 3.1) (layers *.Cu *.Mask)
+      (solder_mask_margin 1.5) (clearance 1.5))
   )
+  (module footprint-lib:MountingHole_3.1mm_M3,rpi_like locked (layer F.Cu)
+    (at 86 66)
+    (descr "Mounting Hole 2.7mm, no annular, M2.5")
+    (tags "mounting hole 2.7mm no annular m2.5")
+    (attr virtual)
+    (fp_text reference H1 (at 0 -3.7) (layer F.SilkS) hide
+      (effects (font (size 1 1) (thickness 0.15)))
+    )
+    (fp_text value MountingHole (at 0 3.7) (layer F.Fab)
+      (effects (font (size 1 1) (thickness 0.15)))
+    )
+    (fp_circle (center 0 0) (end 1.905 0) (layer B.Mask) (width 1.2))
+    (fp_circle (center 0 0) (end 1.905 0) (layer F.Mask) (width 1.2))
+    (fp_circle (center 0 0) (end 2.95 0) (layer F.CrtYd) (width 0.05))
+    (fp_circle (center 0 0) (end 2.7 0) (layer Cmts.User) (width 0.15))
+    (pad "" np_thru_hole circle (at 0 0) (size 3.1 3.1) (drill 3.1) (layers *.Cu *.Mask)
+      (solder_mask_margin 1.5) (clearance 1.5))
+  )
+  (gr_arc (start 4 66) (end 1 66) (angle -90) (layer Dwgs.User) (width 0.15))
+  (gr_arc (start 4 4) (end 4 1) (angle -90) (layer Dwgs.User) (width 0.15))
+  (gr_arc (start 86 4) (end 89 4) (angle -90) (layer Dwgs.User) (width 0.15))
+  (gr_arc (start 86 66) (end 86 69) (angle -90) (layer Dwgs.User) (width 0.15))
+  (gr_arc (start 86 66) (end 86 70) (angle -90) (layer Edge.Cuts) (width 0.15))
+  (gr_arc (start 86 4) (end 90 4) (angle -90) (layer Edge.Cuts) (width 0.15))
+  (gr_arc (start 4 4) (end 4 0) (angle -90) (layer Edge.Cuts) (width 0.15))
+  (gr_arc (start 4 66) (end 0 66) (angle -90) (layer Edge.Cuts) (width 0.15))
+  (gr_text "PCB breadboard\n90 x 70" (at 82 66) (layer F.SilkS)
+    (effects (font (size 1 1) (thickness 0.15)) (justify right))
+  )
+  (gr_line (start 1 66) (end 1 4) (layer Dwgs.User) (width 0.15))
+  (gr_line (start 86 69) (end 4 69) (layer Dwgs.User) (width 0.15))
+  (gr_line (start 89 4) (end 89 66) (layer Dwgs.User) (width 0.15))
+  (gr_line (start 4 1) (end 86 1) (layer Dwgs.User) (width 0.15))
+  (gr_line (start 4 0) (end 86 0) (layer Edge.Cuts) (width 0.15))
+  (gr_line (start 90 4) (end 90 66) (layer Edge.Cuts) (width 0.15))
+  (gr_line (start 4 70) (end 86 70) (layer Edge.Cuts) (width 0.15))
+  (gr_line (start 0 4) (end 0 66) (layer Edge.Cuts) (width 0.15))
 )
