File: 7_by_9_breadboard-tryout/kicad/7_by_9_breadboard-tryout.sch (KiCad schematic (older format))
At the start: 0 parts

Commit message: update basically done,
Parts:
- added H1, H2, H3, H4: MountingHole, footprint-lib:MountingHole_3.1mm_M3,rpi_like, symbol Mechanical:MountingHole
Changed lines of the file:
@@
 Text Notes 700  900  0    50   ~ 0
 helloworld
+$Comp
+L Mechanical:MountingHole H1
+U 1 1 5F3F8107
+P 700 2550
+F 0 "H1" H 800 2596 50  0000 L CNN
+F 1 "MountingHole" H 800 2505 50  0000 L CNN
+F 2 "footprint-lib:MountingHole_3.1mm_M3,rpi_like" H 700 2550 50  0001 C CNN
+F 3 "~" H 700 2550 50  0001 C CNN
+	1    700  2550
+	1    0    0    -1
+$EndComp
+$Comp
+L Mechanical:MountingHole H2
+U 1 1 5F3F85EB
+P 700 2750
+F 0 "H2" H 800 2796 50  0000 L CNN
+F 1 "MountingHole" H 800 2705 50  0000 L CNN
+F 2 "footprint-lib:MountingHole_3.1mm_M3,rpi_like" H 700 2750 50  0001 C CNN
+F 3 "~" H 700 2750 50  0001 C CNN
+	1    700  2750
+	1    0    0    -1
+$EndComp
+$Comp
+L Mechanical:MountingHole H3
+U 1 1 5F3F87A6
+P 700 2950
+F 0 "H3" H 800 2996 50  0000 L CNN
+F 1 "MountingHole" H 800 2905 50  0000 L CNN
+F 2 "footprint-lib:MountingHole_3.1mm_M3,rpi_like" H 700 2950 50  0001 C CNN
+F 3 "~" H 700 2950 50  0001 C CNN
+	1    700  2950
+	1    0    0    -1
+$EndComp
+$Comp
+L Mechanical:MountingHole H4
+U 1 1 5F3F8870
+P 700 3150
+F 0 "H4" H 800 3196 50  0000 L CNN
+F 1 "MountingHole" H 800 3105 50  0000 L CNN
+F 2 "footprint-lib:MountingHole_3.1mm_M3,rpi_like" H 700 3150 50  0001 C CNN
+F 3 "~" H 700 3150 50  0001 C CNN
+	1    700  3150
+	1    0    0    -1
+$EndComp
 $EndSCHEMATC
